File: klima_steuergeraet/klima_steuergeraet.kicad_sch (KiCad schematic)
At the start: 8 parts, among them J1 Screw_Terminal_01x18

Commit message: from uter
Parts:
- added D?: TEST_LED (red), symbol Device:LED
- added J? (x2): Screw_Terminal_01x02, symbol Connector:Screw_Terminal_01x02
- added J? (x2): Conn_01x19, symbol Connector_Generic:Conn_01x19
- added Q?: Q_NMOS_SGD, symbol Device:Q_NMOS_SGD
Connections:
- net SVP (gelb) is gone; now on net GND: J1.3 (Pin_3)
- net 3v3 (weiß): now also J?.1 (Pin_1)
- net GND: now also J?.19 (Pin_19), J?.3 (Pin_3)
- net P16 (grün): now also J?.8 (Pin_8)
- net P17 (braun): now also J?.9 (Pin_9)
- net P18 (grün): now also J?.11 (Pin_11)
- net P19 (gelb): now also J?.12 (Pin_12)
- net P23 (braun): now also J?.18 (Pin_18)
- net P34 (weiß): now also J?.5 (Pin_5)
- net P5 (weiß): now also J?.10 (Pin_10)
- net 5v (gelb): now reaches J1.5 (Pin_5), J1.7 (Pin_7)
- net 5v (gelb): now also J?.19 (Pin_19)
- new net: D?.1 (K), J?.14 (Pin_14)
- new net: D?.2 (A), J?.15 (Pin_15)
- new net: J?.1 (Pin_1), Q?.3 (D)
- new net: J?.1 (Pin_1), J?.2 (Pin_2)
- new net: J?.2 (Pin_2), Q?.1 (S)
- new net P22 (grün): J?.17 (Pin_17), Q?.2 (G)
Other:
- company: (none) -> Kerls Bunker
- title: (none) -> Klimagerät Manta B ESP32
- moved on the sheet: J1, R?
